File: buck-converter-automotive.kicad_sch (KiCad schematic)
At the start: 36 parts, among them J1 12V, J2 5V, U1 MAX17574

Commit message: Make some parts as DNP
Parts:
- C11, R4: now not fitted
Changed lines of the file:
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@@
 		(in_bom yes)
 		(on_board yes)
-		(dnp no)
+		(dnp yes)
 		(property "Reference" "C11"
 			(at 203.2 64.77 90)
@@
 		(in_bom yes)
 		(on_board yes)
-		(dnp no)
+		(dnp yes)
 		(property "Reference" "R4"
 			(at 149.86 67.31 90)
